File: hardware/HMIFeatherWing/kicad_source/HMIFeatherWing.kicad_pcb (KiCad board)
At the start: 2 copper layers, 72 x 30 mm, 25 parts, among them CN1 ARDUINO_MKR, Q1 2N7002, SW1 ALPS_SKRH, SW6 TAST_VER

Commit message: made schematic and layout
Parts:
- CN1: value ARDUINO_MKR -> ADAFRUIT_FEATHER; footprint MODULE_compute:ARDUINO_MKR_HOLES -> MODULE_compute:ADAFRUIT_FEATHER_HOLES
- moved CN1 14.0 mm to (76.0, 96.0)
- moved SW6 2.60 mm to (60.0, 84.5)
Connections:
- CN1 pad 1: Net-(CN1-Pad1) -> /RESET
- CN1 pad 10: /DIS_RESET -> (no net)
- CN1 pad 11: Net-(CN1-Pad11) -> /DIS_CLK
- CN1 pad 12: Net-(CN1-Pad12) -> /DIS_SI
- CN1 pad 16: /DIS_CS -> GND
- CN1 pad 17: /DIS_SI -> (no net)
- CN1 pad 18: /DIS_CLK -> (no net)
- CN1 pad 2: /KEYPAD_A0 -> +3V3
- CN1 pad 22: Net-(CN1-Pad22) -> /DIS_RESET
- CN1 pad 23: Net-(CN1-Pad23) -> /DIS_A0
- CN1 pad 24: /RESET -> /DISPLAY_BL
- CN1 pad 25: GND -> /DIS_CS
- CN1 pad 26: +3V3 -> (no net)
- CN1 pad 4: Net-(CN1-Pad4) -> GND
- CN1 pad 5: Net-(CN1-Pad5) -> /KEYPAD_A0
- CN1 pad 8: /DISPLAY_BL -> (no net)
- CN1 pad 9: /DIS_A0 -> (no net)
Routing:
- net /DIS_CS: track 37.6 -> 5.44 mm
- net /DISPLAY_BL: track 28.4 -> 58.5 mm
- net /DIS_A0: track 34.9 -> 5.44 mm, vias 1 -> 0
- net /DIS_RESET: track 39.0 -> 12.1 mm, vias 1 -> 0
- net +3V3: track 82.8 -> 93.6 mm, vias 2 -> 3
- net /KEYPAD_A0: track 27.9 -> 35.1 mm
- net GND: track 28.6 -> 23.3 mm, vias 6 -> 7
- net /DIS_SI: track 23.9 -> 28.9 mm
- net /DIS_CLK: track 33.2 -> 28.4 mm
- net /RESET: track 28.6 -> 30.5 mm
Other:
- board text added: "HMIFeatherWing"
- board text removed: "MKR HMI"

Commit message: checked pins to fit to other feather wings, used smaller reset, corrected joystick orientation, connected backlight, made board smaller, finished layout
Parts:
- removed SW6: TAST_VER, mechanical-switches:WE_430182050816
- added G***: generationmake_logo, labels:generationmake_logo, B.Cu at (100.8, 102.3)
- added G***: generationmake_small_solder, labels:generationmake_small_solder, F.Cu at (62.5, 92.2)
- added R10: 0R, resistors:R_0603, F.Cu at (72.2, 102.4)
- added R6: DNI, resistors:R_0603, F.Cu at (70.5, 102.4)
- added SW2: SW_PUSH, mechanical-switches:smd_push, F.Cu at (63.2, 83.9)
- moved R3 15.4 mm to (64.6, 102.3)
- moved R5 9.50 mm to (57.6, 92.0), turned to 90 degrees
- moved R4 7.96 mm to (58.6, 102.3)
- moved C11 7.01 mm to (84.9, 83.8)
- moved R2 6.44 mm to (70.2, 95.6)
- moved R1 6.43 mm to (69.9, 100.0), turned to 0 degrees
- moved SW1 5.10 mm to (58.0, 98.0), turned to 0 degrees
- moved CN1 5.00 mm to (81.0, 96.0)
Connections:
- CN1 pad 10: (no net) -> /KEYPAD_A0_5
- CN1 pad 13: Net-(CN1-Pad13) -> (no net)
- CN1 pad 14: Net-(CN1-Pad14) -> (no net)
- CN1 pad 15: Net-(CN1-Pad15) -> (no net)
- CN1 pad 16: GND -> (no net)
- CN1 pad 19: Net-(CN1-Pad19) -> (no net)
- CN1 pad 20: Net-(CN1-Pad20) -> (no net)
- CN1 pad 21: Net-(CN1-Pad21) -> (no net)
- CN1 pad 22: /DIS_RESET -> (no net)
- CN1 pad 23: /DIS_A0 -> (no net)
- CN1 pad 24: /DISPLAY_BL -> (no net)
- CN1 pad 25: /DIS_CS -> /DISPLAY_BL
- CN1 pad 27: Net-(CN1-Pad27) -> (no net)
- CN1 pad 28: Net-(CN1-Pad28) -> (no net)
- CN1 pad 3: Net-(CN1-Pad3) -> (no net)
- CN1 pad 5: /KEYPAD_A0 -> /KEYPAD_A0_0
- CN1 pad 6: Net-(CN1-Pad6) -> /DIS_CS
- CN1 pad 7: Net-(CN1-Pad7) -> /DIS_RESET
- CN1 pad 8: (no net) -> /DIS_A0
- DIS2 pad 1: +5V -> +3V3
- DIS2 pad 20: +5V -> +3V3
Routing:
- net +5V: track 50.3 -> 0.00 mm
- net /DIS_CS: track 5.44 -> 29.5 mm
- net /KEYPAD_A0: track 35.1 -> 12.2 mm
- net /DIS_A0: track 5.44 -> 25.7 mm
- net +3V3: track 93.6 -> 111.8 mm, vias 3 -> 2
- net /KEYPAD_A0_5: track 0.00 -> 16.3 mm
- net /DIS_RESET: track 12.1 -> 26.5 mm
- net /BUTTON_DOWN: track 18.4 -> 11.0 mm
- net GND: track 23.3 -> 27.0 mm, vias 7 -> 17
- net /KEYPAD_A0_0: track 0.00 -> 3.68 mm
- net /RESET: track 30.5 -> 27.3 mm, vias 0 -> 1
- net /DISPLAY_BL: track 58.5 -> 56.7 mm
- net /DIS_CLK: track 28.4 -> 29.9 mm
- net /BUTTON_SELECT: track 4.88 -> 3.49 mm
- net /BUTTON_UP: track 19.8 -> 18.5 mm
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Other:
- board size 72 x 30 mm -> 67 x 30 mm
- board text removed: "ArduHMI"
